Commit message: finished and tested trajectory generation + improved comments on tasks

File: examples/05-two_hand_two_robots_object_movement/panda_arm.urdf (robot description, URDF)
Before this commit: robot panda, 8 links, 7 joints
Links:
- link link7: mass 0.5 -> 1.8

File: examples/05-two_hand_two_robots_object_movement/panda_arm_hand.urdf (robot description, URDF)
Before this commit: robot panda_hand, 10 links, 9 joints
Links:
- link link4: geometry collision mesh filename=../../../../examples/models/panda/meshes/collision/link4.obj; visual mesh filename=../../../../examples/models/panda/meshes/visual/link4.obj
Joints:
- joint finger_joint2: mimic joint=finger_joint1 -> (none)
